Commit message: renaming of the joints to not have a "->" which messed with the xml file

File: config/dexarm.ros2_control.xacro (robot description, xacro)
@@ -28,15 +28,15 @@
                 <state_interface name="velocity"/>
             </joint>
-            <joint name="B_Rot->In_1">
+            <joint name="B_Rot-In_1">
                 <command_interface name="position"/>
                 <state_interface name="position">
-                  <param name="initial_value">${initial_positions['B_Rot->In_1']}</param>
+                  <param name="initial_value">${initial_positions['B_Rot-In_1']}</param>
                 </state_interface>
                 <state_interface name="velocity"/>
             </joint>
-            <joint name="Join->In_2">
+            <joint name="Join-In_2">
                 <command_interface name="position"/>
                 <state_interface name="position">
-                  <param name="initial_value">${initial_positions['Join->In_2']}</param>
+                  <param name="initial_value">${initial_positions['Join-In_2']}</param>
                 </state_interface>
                 <state_interface name="velocity"/>

File: urdf/dexarm.xacro (robot description, xacro)
@@ -9,5 +9,4 @@
     <xacro:arg name="use_gripper" default="false" /> <!-- gripper or vacuum suction -->
     <xacro:arg name="use_vacuum_suction" default="true" />
-    <!-- ROS Control related parameters-->
     <!-- Constants for robot dimensions -->
     <xacro:property name="PI" value="3.1415926535897931"/>
@@ -208,8 +207,8 @@
     </link>
     <xacro:if value="$(arg use_vacuum_suction)">
-        <xacro include="suction_gripper.xacro"/>
+        <xacro:include filename="$(find dexarm_description)/urdf/suction_gripper.xacro"/>
     </xacro:if>
     <xacro:if value="$(arg use_gripper)">
-        <xacro include="soft_gripper.xacro"/>
+        <xacro:include filename="$(find dexarm_description)/urdf/soft_gripper.xacro"/>
     </xacro:if>
     <!-- <joint name="EE-Suction" type="fixed">

File: urdf/soft_gripper.xacro (robot description, xacro)
@@ -1,368 +1,371 @@
-<joint name="EE-GripperMount" type="fixed">
-    <parent link="EE" />
-    <child link="GripperMount" />
-    <limit effort="30" lower="-0.6" upper="1.2" velocity="1.74533" />
-    <origin xyz="0 -0.05 0.01" rpy="0 0 0"/>
-    <axis xyz="1 0 0" />
-</joint>
-<link name="GripperMount">
-    <visual>
-      <origin xyz="-0.077 -0.134 -0.003" rpy="0 3.14 1.57" />
-      <geometry>
-        <mesh filename="package://dexarm_description/urdf/STL/M02-GripperMount.stl" scale="0.001 0.001 0.001"/>
-      </geometry>
-    </visual>
-    <collision>
-      <origin xyz="-0.077 -0.134 -0.003" rpy="0 3.14 1.57"/>
-      <geometry>
-        <mesh filename="package://dexarm_description/urdf/STL/M02-GripperMount.stl" scale="0.001 0.001 0.001"/>
-      </geometry>
-    </collision>
-</link>
-<joint name="GripperMount-GripperAxis" type="continuous">
-    <parent link="GripperMount" />
-    <child link="GripperAxis" />
-    <limit effort="30" velocity="1.74533" />
-    <origin xyz="-0.002 -0.06 0.0" rpy="0 0 0"/>
-    <axis xyz="0 0 1" />
-</joint>
-<link name="GripperAxis">
-    <visual>
-        <origin xyz="-0.075 -0.075 -0.000" rpy="0 3.14 1.57" />
-        <geometry>
-        <mesh filename="package://dexarm_description/urdf/STL/M02-GripperAxis.stl" scale="0.001 0.001 0.001"/>
-        </geometry>
-    </visual>
-    <collision>
-        <origin xyz="-0.075 -0.075 -0.000" rpy="0 3.14 1.57"/>
-        <geometry>
-        <mesh filename="package://dexarm_description/urdf/STL/M02-GripperAxis.stl" scale="0.001 0.001 0.001"/>
-        </geometry>
-    </collision>
-</link>
-<joint name="GripperAxis-GripperFingerA1" type="fixed">
-    <parent link="GripperAxis" />
-    <child link="GripperFingerA1" />
-    <limit effort="30" velocity="1.74533" />
-    <origin xyz="-0.020 0.00 -0.042" rpy="0 0 0"/>
-    <axis xyz="0 0 1" />
-</joint>
-<link name="GripperFingerA1">
-    <visual>
-        <origin xyz="-0.054 -0.075 0.036" rpy="0.0 3.14 1.57" />
+<?xml version="1.0"?>
+<robot>
+    <joint name="EE-GripperMount" type="fixed">
+        <parent link="EE" />
+        <child link="GripperMount" />
+        <limit effort="30" lower="-0.6" upper="1.2" velocity="1.74533" />
+        <origin xyz="0 -0.05 0.01" rpy="0 0 0"/>
+        <axis xyz="1 0 0" />
+    </joint>
+    <link name="GripperMount">
+        <visual>
+        <origin xyz="-0.077 -0.134 -0.003" rpy="0 3.14 1.57" />
+        <geometry>
+            <mesh filename="package://dexarm_description/urdf/STL/M02-GripperMount.stl" scale="0.001 0.001 0.001"/>
+        </geometry>
+        </visual>
+        <collision>
+        <origin xyz="-0.077 -0.134 -0.003" rpy="0 3.14 1.57"/>
+        <geometry>
+            <mesh filename="package://dexarm_description/urdf/STL/M02-GripperMount.stl" scale="0.001 0.001 0.001"/>
+        </geometry>
+        </collision>
+    </link>
+    <joint name="GripperMount-GripperAxis" type="continuous">
+        <parent link="GripperMount" />
+        <child link="GripperAxis" />
+        <limit effort="30" velocity="1.74533" />
+        <origin xyz="-0.002 -0.06 0.0" rpy="0 0 0"/>
+        <axis xyz="0 0 1" />
+    </joint>
+    <link name="GripperAxis">
+        <visual>
+            <origin xyz="-0.075 -0.075 -0.000" rpy="0 3.14 1.57" />
+            <geometry>
+            <mesh filename="package://dexarm_description/urdf/STL/M02-GripperAxis.stl" scale="0.001 0.001 0.001"/>
+            </geometry>
+        </visual>
+        <collision>
+            <origin xyz="-0.075 -0.075 -0.000" rpy="0 3.14 1.57"/>
+            <geometry>
+            <mesh filename="package://dexarm_description/urdf/STL/M02-GripperAxis.stl" scale="0.001 0.001 0.001"/>
+            </geometry>
+        </collision>
+    </link>
+    <joint name="GripperAxis-GripperFingerA1" type="fixed">
+        <parent link="GripperAxis" />
+        <child link="GripperFingerA1" />
+        <limit effort="30" velocity="1.74533" />
+        <origin xyz="-0.020 0.00 -0.042" rpy="0 0 0"/>
+        <axis xyz="0 0 1" />
+    </joint>
+    <link name="GripperFingerA1">
+        <visual>
+            <origin xyz="-0.054 -0.075 0.036" rpy="0.0 3.14 1.57" />
+            <geometry>
+                <mesh filename="package://dexarm_description/urdf/STL/M02-GripperFinger1.stl" scale="0.001 0.001 0.001"/>
+            </geometry>
+        </visual>
+        <collision>
+            <origin xyz="-0.054 -0.075 0.036" rpy="0.0 3.14 1.57" />
+            <geometry>
+                <mesh filename="package://dexarm_description/urdf/STL/M02-GripperFinger1.stl" scale="0.001 0.001 0.001"/>
+            </geometry>
+            </collision>
+    </link>
+    <link name="GripperFingerA2">
+        <visual>
+        <origin xyz="-0.057 -0.075 0.0440" rpy="0.0 3.14 1.57" />
+        <geometry>
+            <mesh filename="package://dexarm_description/urdf/STL/M02-GripperFinger2.stl" scale="0.001 0.001 0.001"/>
+        </geometry>
+        </visual>
+        <collision>
+        <origin xyz="-0.057 -0.075 0.0440" rpy="0.0 3.14 1.57" />
+        <geometry>
+            <mesh filename="package://dexarm_description/urdf/STL/M02-GripperFinger2.stl" scale="0.001 0.001 0.001"/>
+        </geometry>
+        </collision>
+    </link>
+    <joint name="GripperFingerA1-GripperFingerA2" type="revolute">
+        <parent link="GripperFingerA1" />
+        <child link="GripperFingerA2" />
+        <limit effort="30" lower="-0.3" upper="0.0" velocity="1.74533" />
+        <origin xyz="0.003 0.00 -0.008" rpy="0 0 0"/>
+        <axis xyz="0 1 0" />
+    </joint>
+    <link name="GripperFingerA3">
+        <visual>
+        <origin xyz="-0.0575 -0.075 0.0510" rpy="0.0 3.14 1.57" />
+        <geometry>
+            <mesh filename="package://dexarm_description/urdf/STL/M02-GripperFinger3.stl" scale="0.001 0.001 0.001"/>
+        </geometry>
+        </visual>
+        <collision>
+        <origin xyz="-0.0575 -0.075 0.0510" rpy="0.0 3.14 1.57" />
+        <geometry>
+            <mesh filename="package://dexarm_description/urdf/STL/M02-GripperFinger3.stl" scale="0.001 0.001 0.001"/>
+        </geometry>
+        </collision>
+    </link>
+    <joint name="GripperFingerA2-GripperFingerA3" type="revolute">
+        <parent link="GripperFingerA2" />
+        <child link="GripperFingerA3" />
+        <limit effort="30" lower="-0.3" upper="0.0" velocity="1.74533" />
+        <origin xyz="0.0005 0.00 -0.007" rpy="0 0 0"/>
+        <axis xyz="0 1 0" />
+        <mimic joint="GripperFingerA1-GripperFingerA2" multiplier="1" offset="0" />
+    </joint>
+    <link name="GripperFingerA4">
+        <visual>
+        <origin xyz="-0.0580 -0.075 0.0580" rpy="0.0 3.14 1.57" />
+        <geometry>
+            <mesh filename="package://dexarm_description/urdf/STL/M02-GripperFinger4.stl" scale="0.001 0.001 0.001"/>
+        </geometry>
+        </visual>
+        <collision>
+        <origin xyz="-0.0580 -0.075 0.0580" rpy="0.0 3.14 1.57" />
+        <geometry>
+            <mesh filename="package://dexarm_description/urdf/STL/M02-GripperFinger4.stl" scale="0.001 0.001 0.001"/>
+        </geometry>
+        </collision>
+    </link>
+    <joint name="GripperFingerA3-GripperFingerA4" type="revolute">
+        <parent link="GripperFingerA3" />
+        <child link="GripperFingerA4" />
+        <limit effort="30" lower="-0.3" upper="0.0" velocity="1.74533" />
+        <origin xyz="0.0005 0.00 -0.007" rpy="0 0 0"/>
+        <axis xyz="0 1 0" />
+        <mimic joint="GripperFingerA1-GripperFingerA2" multiplier="1" offset="0" />
+    </joint>
+    <link name="GripperFingerA5">
+        <visual>
+        <origin xyz="-0.0585 -0.075 0.0650" rpy="0.0 3.14 1.57" />
+        <geometry>
+            <mesh filename="package://dexarm_description/urdf/STL/M02-GripperFinger5.stl" scale="0.001 0.001 0.001"/>
+        </geometry>
+        </visual>
+        <collision>
+        <origin xyz="-0.0585 -0.075 0.0650" rpy="0.0 3.14 1.57" />
+        <geometry>
+            <mesh filename="package://dexarm_description/urdf/STL/M02-GripperFinger5.stl" scale="0.001 0.001 0.001"/>
+        </geometry>
+        </collision>
+    </link>
+    <joint name="GripperFingerA4-GripperFingerA5" type="revolute">
+        <parent link="GripperFingerA4" />
+        <child link="GripperFingerA5" />
+        <limit effort="30" lower="-0.3" upper="0.0" velocity="1.74533" />
+        <origin xyz="0.0005 0.00 -0.007" rpy="0 0 0"/>
+        <axis xyz="0 1 0" />
+        <mimic joint="GripperFingerA1-GripperFingerA2" multiplier="1" offset="0" />
+    </joint>
+    <link name="GripperFingerB1">
+        <visual>
+        <origin xyz="-0.038 0.084 0.036" rpy="0.0 3.14 5.76" />
         <geometry>
             <mesh filename="package://dexarm_description/urdf/STL/M02-GripperFinger1.stl" scale="0.001 0.001 0.001"/>
         </geometry>
-    </visual>
-    <collision>
-        <origin xyz="-0.054 -0.075 0.036" rpy="0.0 3.14 1.57" />
+        </visual>
+        <collision>
+        <origin xyz="-0.038 0.084 0.036" rpy="0.0 3.14 5.76" />
         <geometry>
             <mesh filename="package://dexarm_description/urdf/STL/M02-GripperFinger1.stl" scale="0.001 0.001 0.001"/>
         </geometry>
         </collision>
-</link>
-<link name="GripperFingerA2">
-    <visual>
-      <origin xyz="-0.057 -0.075 0.0440" rpy="0.0 3.14 1.57" />
-      <geometry>
-        <mesh filename="package://dexarm_description/urdf/STL/M02-GripperFinger2.stl" scale="0.001 0.001 0.001"/>
-      </geometry>
-    </visual>
-    <collision>
-      <origin xyz="-0.057 -0.075 0.0440" rpy="0.0 3.14 1.57" />
-      <geometry>
-        <mesh filename="package://dexarm_description/urdf/STL/M02-GripperFinger2.stl" scale="0.001 0.001 0.001"/>
-      </geometry>
-    </collision>
-</link>
-<joint name="GripperFingerA1-GripperFingerA2" type="revolute">
-    <parent link="GripperFingerA1" />
-    <child link="GripperFingerA2" />
-    <limit effort="30" lower="-0.3" upper="0.0" velocity="1.74533" />
-    <origin xyz="0.003 0.00 -0.008" rpy="0 0 0"/>
-    <axis xyz="0 1 0" />
-</joint>
-<link name="GripperFingerA3">
-    <visual>
-      <origin xyz="-0.0575 -0.075 0.0510" rpy="0.0 3.14 1.57" />
-      <geometry>
-        <mesh filename="package://dexarm_description/urdf/STL/M02-GripperFinger3.stl" scale="0.001 0.001 0.001"/>
-      </geometry>
-    </visual>
-    <collision>
-      <origin xyz="-0.0575 -0.075 0.0510" rpy="0.0 3.14 1.57" />
-      <geometry>
-        <mesh filename="package://dexarm_description/urdf/STL/M02-GripperFinger3.stl" scale="0.001 0.001 0.001"/>
-      </geometry>
-    </collision>
-</link>
-<joint name="GripperFingerA2-GripperFingerA3" type="revolute">
-    <parent link="GripperFingerA2" />
-    <child link="GripperFingerA3" />
-    <limit effort="30" lower="-0.3" upper="0.0" velocity="1.74533" />
-    <origin xyz="0.0005 0.00 -0.007" rpy="0 0 0"/>
-    <axis xyz="0 1 0" />
-    <mimic joint="GripperFingerA1-GripperFingerA2" multiplier="1" offset="0" />
-</joint>
-<link name="GripperFingerA4">
-    <visual>
-      <origin xyz="-0.0580 -0.075 0.0580" rpy="0.0 3.14 1.57" />
-      <geometry>
-        <mesh filename="package://dexarm_description/urdf/STL/M02-GripperFinger4.stl" scale="0.001 0.001 0.001"/>
-      </geometry>
-    </visual>
-    <collision>
-      <origin xyz="-0.0580 -0.075 0.0580" rpy="0.0 3.14 1.57" />
-      <geometry>
-        <mesh filename="package://dexarm_description/urdf/STL/M02-GripperFinger4.stl" scale="0.001 0.001 0.001"/>
-      </geometry>
-    </collision>
-</link>
-<joint name="GripperFingerA3-GripperFingerA4" type="revolute">
-    <parent link="GripperFingerA3" />
-    <child link="GripperFingerA4" />
-    <limit effort="30" lower="-0.3" upper="0.0" velocity="1.74533" />
-    <origin xyz="0.0005 0.00 -0.007" rpy="0 0 0"/>
-    <axis xyz="0 1 0" />
-    <mimic joint="GripperFingerA1-GripperFingerA2" multiplier="1" offset="0" />
-</joint>
-<link name="GripperFingerA5">
-    <visual>
-      <origin xyz="-0.0585 -0.075 0.0650" rpy="0.0 3.14 1.57" />
-      <geometry>
-        <mesh filename="package://dexarm_description/urdf/STL/M02-GripperFinger5.stl" scale="0.001 0.001 0.001"/>
-      </geometry>
-    </visual>
-    <collision>
-      <origin xyz="-0.0585 -0.075 0.0650" rpy="0.0 3.14 1.57" />
-      <geometry>
-        <mesh filename="package://dexarm_description/urdf/STL/M02-GripperFinger5.stl" scale="0.001 0.001 0.001"/>
-      </geometry>
-    </collision>
-</link>
-<joint name="GripperFingerA4-GripperFingerA5" type="revolute">
-    <parent link="GripperFingerA4" />
-    <child link="GripperFingerA5" />
-    <limit effort="30" lower="-0.3" upper="0.0" velocity="1.74533" />
-    <origin xyz="0.0005 0.00 -0.007" rpy="0 0 0"/>
-    <axis xyz="0 1 0" />
-    <mimic joint="GripperFingerA1-GripperFingerA2" multiplier="1" offset="0" />
-</joint>
-<link name="GripperFingerB1">
-    <visual>
-      <origin xyz="-0.038 0.084 0.036" rpy="0.0 3.14 5.76" />
-      <geometry>
-        <mesh filename="package://dexarm_description/urdf/STL/M02-GripperFinger1.stl" scale="0.001 0.001 0.001"/>
-      </geometry>
-    </visual>
-    <collision>
-      <origin xyz="-0.038 0.084 0.036" rpy="0.0 3.14 5.76" />
-      <geometry>
-        <mesh filename="package://dexarm_description/urdf/STL/M02-GripperFinger1.stl" scale="0.001 0.001 0.001"/>
-      </geometry>
-    </collision>
-</link>
-<joint name="GripperAxis-GripperFingerB1" type="fixed">
-    <parent link="GripperAxis" />
-    <child link="GripperFingerB1" />
-    <limit effort="30" velocity="1.74533" />
-    <origin xyz="0.010 0.018 -0.042" rpy="0 0 0.0"/>
-    <axis xyz="0 0 1" />
-</joint>
-<link name="GripperFingerB2">
-    <visual>
-      <origin xyz="0.0616 0.0710 0.044" rpy="0.0 3.14 4.66" />
-      <geometry>
-        <mesh filename="package://dexarm_description/urdf/STL/M02-GripperFinger2.stl" scale="0.001 0.001 0.001"/>
-      </geometry>
-    </visual>
-    <collision>
-      <origin xyz="0.0616 0.0710 0.044" rpy="0.0 3.14 4.66" />
-      <geometry>
-        <mesh filename="package://dexarm_description/urdf/STL/M02-GripperFinger2.stl" scale="0.001 0.001 0.001"/>
-      </geometry>
-    </collision>
-</link>
-<joint name="GripperFingerB1-GripperFingerB2" type="revolute">
-    <parent link="GripperFingerB1" />
-    <child link="GripperFingerB2" />
-    <limit effort="30" lower="0.0" upper="0.3" velocity="1.74533" />
-    <origin xyz="-0.003 -0.003 -0.008" rpy="0 0 1.1"/>
-    <axis xyz="0 1 0" />
-    <mimic joint="GripperFingerA1-GripperFingerA2" multiplier="-1" offset="0" />
-</joint>
-<link name="GripperFingerB3">
-    <visual>
-      <origin xyz="0.0616 0.0710 0.050" rpy="0.0 3.14 4.66" />
-      <geometry>
-        <mesh filename="package://dexarm_description/urdf/STL/M02-GripperFinger3.stl" scale="0.001 0.001 0.001"/>
-      </geometry>
-    </visual>
-    <collision>
-      <origin xyz="0.0616 0.0710 0.050" rpy="0.0 3.14 4.66" />
-      <geometry>
-        <mesh filename="package://dexarm_description/urdf/STL/M02-GripperFinger3.stl" scale="0.001 0.001 0.001"/>
-      </geometry>
-    </collision>
-</link>
-<joint name="GripperFingerB2-GripperFingerB3" type="revolute">
-    <parent link="GripperFingerB2" />
-    <child link="GripperFingerB3" />
-    <limit effort="30" lower="0" upper="0.3" velocity="1.74533" />
-    <origin xyz="-0.000 -0.000 -0.006" rpy="0 0 0.0"/>
-    <axis xyz="0 1 0" />
-    <mimic joint="GripperFingerA1-GripperFingerA2" multiplier="-1" offset="0" />
-</joint>
-<link name="GripperFingerB4">
-    <visual>
-      <origin xyz="0.0611 0.0710 0.057" rpy="0.0 3.14 4.66" />
-      <geometry>
-        <mesh filename="package://dexarm_description/urdf/STL/M02-GripperFinger4.stl" scale="0.001 0.001 0.001"/>
-      </geometry>
-    </visual>
-    <collision>
-      <origin xyz="0.0611 0.0710 0.057" rpy="0.0 3.14 4.66" />
-      <geometry>
-        <mesh filename="package://dexarm_description/urdf/STL/M02-GripperFinger4.stl" scale="0.001 0.001 0.001"/>
-      </geometry>
-    </collision>
-</link>
-<joint name="GripperFingerB3-GripperFingerB4" type="revolute">
-    <parent link="GripperFingerB3" />
-    <child link="GripperFingerB4" />
-    <limit effort="30" lower="0." upper="0.3" velocity="1.74533" />
-    <origin xyz="0.0005 0.00 -0.007" rpy="0 0 0.0"/>
-    <axis xyz="0 1 0" />
-    <mimic joint="GripperFingerA1-GripperFingerA2" multiplier="-1" offset="0" />
-</joint>
-<link name="GripperFingerB5">
-    <visual>
-      <origin xyz="0.0607 0.0710 0.0641" rpy="0.0 3.14 4.66" />
-      <geometry>
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
File: urdf/suction_gripper.xacro (robot description, xacro)
@@ -1,21 +1,24 @@
-<joint name="EE->Suction" type="fixed">
-    <parent link="EE" />
-    <child link="Suction" />
-    <limit effort="30" lower="-0.6" upper="1.2" velocity="1.74533" />
-    <origin xyz="0 -0.05 0.01" rpy="0 0 0"/>
-    <axis xyz="1 0 0" />
-</joint>
-<link name="Suction">
-    <visual>
-        <origin xyz="-0.077 -0.134 -0.003" rpy="0 3.14 1.57" />
-        <geometry>
-        <mesh filename="package://dexarm_description/urdf/STL/M01-Suction.stl" scale="0.001 0.001 0.001"/>
-        </geometry>
-    </visual>
-    <collision>
-        <origin xyz="-0.077 -0.134 -0.003" rpy="0 3.14 1.57"/>
-        <geometry>
-        <mesh filename="package://dexarm_description/urdf/STL/M01-Suction.stl" scale="0.001 0.001 0.001"/>
-        </geometry>
-    </collision>
-</link>
+<?xml version="1.0"?>
+<robot>
+    <joint name="EE-Suction" type="fixed">
+        <parent link="EE" />
+        <child link="Suction" />
+        <limit effort="30" lower="-0.6" upper="1.2" velocity="1.74533" />
+        <origin xyz="0 -0.05 0.01" rpy="0 0 0"/>
+        <axis xyz="1 0 0" />
+    </joint>
+    <link name="Suction">
+        <visual>
+            <origin xyz="-0.077 -0.134 -0.003" rpy="0 3.14 1.57" />
+            <geometry>
+            <mesh filename="package://dexarm_description/urdf/STL/M01-Suction.stl" scale="0.001 0.001 0.001"/>
+            </geometry>
+        </visual>
+        <collision>
+            <origin xyz="-0.077 -0.134 -0.003" rpy="0 3.14 1.57"/>
+            <geometry>
+            <mesh filename="package://dexarm_description/urdf/STL/M01-Suction.stl" scale="0.001 0.001 0.001"/>
+            </geometry>
+        </collision>
+    </link>
+</robot>
