Commit message: Delete virtual joint link

File: urdf/dexarm.xacro (robot description, xacro)
@@ -18,9 +18,9 @@
     <!-- <xacro:include filename="$(find dexarm_moveit_config)/config/dexarm.ros2_control.xacro" /> -->
     <!-- For simulation  -->
-    <link name="world"/>
+    <!-- <link name="world"/>
     <joint name="fixed" type="fixed">
         <parent link="world"/>
         <child link="B_Fix"/>
-    </joint>
+    </joint> -->
     <link name="B_Fix">
         <visual>

Commit message: move some files from the moveit_config to the description package for launch purposes

File: urdf/dexarm.xacro (robot description, xacro)
@@ -13,14 +13,25 @@
     <xacro:arg name="use_fake_hardware" default="true" />
     <xacro:arg name="fake_sensor_commands" default="false" />
+    <!-- dexarm_description/urdf/initial_positions.yaml -->
+    <!-- <xacro:arg name="initial_positions_file" default="$(find dexarm_description)/urdf/initial_positions.yaml)" /> -->
+    <xacro:arg name="initial_positions_file" default="/home/luke/dexarm_ws/src/dexarm_description/urdf/initial_positions.yaml" />
+    <!-- convert to property to use substitution in function -->
+   <!-- <xacro:property name="initial_positions_file" default="$(arg initial_positions_file)"/> -->
     <!-- Import all Gazebo-customization elements, including Gazebo colors -->
-    <xacro:include filename="$(find dexarm_description)/urdf/dexarm.gazebo" />
+    <xacro:if value="$(arg is_simulation)">
+        <xacro:include filename="$(find dexarm_description)/urdf/dexarm.gazebo" />
+    </xacro:if>
     <!-- Import control_xacro -->
-    <!-- <xacro:include filename="$(find dexarm_moveit_config)/config/dexarm.ros2_control.xacro" /> -->
+    <!-- <xacro:include filename="/home/luke/dexarm_ws/src/dexarm_moveit_config/config/dexarm.ros2_control.xacro" /> -->
+    <xacro:include filename="dexarm.ros2_control.xacro" />
+    <xacro:dexarm_ros2_control name="dexarm" initial_positions_file="$(arg initial_positions_file)"/>
+    <!-- <xacro:dexarm_ros2_control name="dexarm" initial_positions_file="${xacro.load_yaml($(find dexarm_description)/urdf/inital_positions.yaml)}"/> -->
+    <!-- <xacro:dexarm_ros2_control name="dexarm" initial_positions_file="${xacro.load_yaml(initial_positions_file)}"/> -->
     <!-- For simulation  -->
-    <!-- <link name="world"/>
+    <link name="world"/>
     <joint name="fixed" type="fixed">
         <parent link="world"/>
         <child link="B_Fix"/>
-    </joint> -->
+    </joint>
     <link name="B_Fix">
         <visual>

Commit message: make the gripper changeable via xacro

File: urdf/dexarm.xacro (robot description, xacro)
@@ -2,4 +2,12 @@
 <!-- Revolute-Revolute Manipulator -->
 <robot name="dexarm" xmlns:xacro="http://www.ros.org/wiki/xacro">
+    <!-- ARGUMENTS -->
+    <xacro:arg name="is_simulation" default="true" />
+    <xacro:arg name="use_fake_hardware" default="true" />
+    <xacro:arg name="fake_sensor_commands" default="false" />
+    <xacro:arg name="prefix" default="" />
+    <xacro:arg name="use_gripper" default="false" /> <!-- gripper or vacuum suction -->
+    <xacro:arg name="use_vacuum_suction" default="true" />
+    <!-- ROS Control related parameters-->
     <!-- Constants for robot dimensions -->
     <xacro:property name="PI" value="3.1415926535897931"/>
@@ -9,13 +17,9 @@
     <xacro:property name="height2" value="1" /> <!-- Link 2 -->
     <xacro:property name="height3" value="1" /> <!-- Link 3 -->
-    <!-- ARGUMENTS -->
-    <xacro:arg name="is_simulation" default="true" />
-    <xacro:arg name="use_fake_hardware" default="true" />
-    <xacro:arg name="fake_sensor_commands" default="false" />
     <!-- dexarm_description/urdf/initial_positions.yaml -->
     <!-- <xacro:arg name="initial_positions_file" default="$(find dexarm_description)/urdf/initial_positions.yaml)" /> -->
-    <xacro:arg name="initial_positions_file" default="/home/luke/dexarm_ws/src/dexarm_description/urdf/initial_positions.yaml" />
+    <xacro:arg name="initial_positions_file" default="$(find dexarm_description)/config/initial_positions.yaml" />
     <!-- convert to property to use substitution in function -->
-   <!-- <xacro:property name="initial_positions_file" default="$(arg initial_positions_file)"/> -->
+    <!-- <xacro:property name="initial_positions_file" default="$(arg initial_positions_file)"/> -->
     <!-- Import all Gazebo-customization elements, including Gazebo colors -->
     <xacro:if value="$(arg is_simulation)">
@@ -24,5 +28,5 @@
     <!-- Import control_xacro -->
     <!-- <xacro:include filename="/home/luke/dexarm_ws/src/dexarm_moveit_config/config/dexarm.ros2_control.xacro" /> -->
-    <xacro:include filename="dexarm.ros2_control.xacro" />
+    <xacro:include filename="$(find dexarm_description)/config/dexarm.ros2_control.xacro" />
     <xacro:dexarm_ros2_control name="dexarm" initial_positions_file="$(arg initial_positions_file)"/>
     <!-- <xacro:dexarm_ros2_control name="dexarm" initial_positions_file="${xacro.load_yaml($(find dexarm_description)/urdf/inital_positions.yaml)}"/> -->
@@ -85,5 +89,5 @@
         </inertial>
     </link>
-    <joint name="B_Rot->In_1" type="revolute">
+    <joint name="B_Rot-In_1" type="revolute">
         <parent link="B_Rot" />
         <child link="In_1" />
@@ -114,5 +118,5 @@
         </inertial>
     </link>
-    <joint name="In_1->Join" type="revolute">
+    <joint name="In_1-Join" type="revolute">
         <parent link="In_1" />
         <child link="Join" />
@@ -144,5 +148,5 @@
         </inertial>
     </link>
-    <joint name="Join->In_2" type="revolute">
+    <joint name="Join-In_2" type="revolute">
         <parent link="Join" />
         <child link="In_2" />
@@ -173,5 +177,5 @@
         </inertial>
     </link>
-    <joint name="In_2->EE" type="revolute">
+    <joint name="In_2-EE" type="revolute">
         <parent link="In_2" />
         <child link="EE" />
@@ -203,5 +207,11 @@
         </inertial>
     </link>
-    <joint name="EE->Suction" type="fixed">
+    <xacro:if value="$(arg use_vacuum_suction)">
+        <xacro include="suction_gripper.xacro"/>
+    </xacro:if>
+    <xacro:if value="$(arg use_gripper)">
+        <xacro include="soft_gripper.xacro"/>
+    </xacro:if>
+    <!-- <joint name="EE-Suction" type="fixed">
         <parent link="EE" />
         <child link="Suction" />
@@ -231,4 +241,4 @@
                 izz="${mass / 12.0 * (width*width + width*width)}"/>
         </inertial>
-    </link>
+    </link> -->
 </robot>

Commit message: move some of the moveit setup config files into this package

File: urdf/dexarm.xacro (robot description, xacro)
@@ -29,12 +29,10 @@
     <xacro:include filename="$(find dexarm_description)/config/dexarm.ros2_control.xacro" />
     <xacro:dexarm_ros2_control name="dexarm" initial_positions_file="$(arg initial_positions_file)"/>
-    <!-- <xacro:dexarm_ros2_control name="dexarm" initial_positions_file="${xacro.load_yaml($(find dexarm_description)/urdf/inital_positions.yaml)}"/> -->
-    <!-- <xacro:dexarm_ros2_control name="dexarm" initial_positions_file="${xacro.load_yaml(initial_positions_file)}"/> -->
     <!-- For simulation  -->
-    <link name="world"/>
+    <!-- <link name="world"/>
     <joint name="fixed" type="fixed">
         <parent link="world"/>
         <child link="B_Fix"/>
-    </joint>
+    </joint>  -->
     <link name="B_Fix">
         <visual>
@@ -123,5 +121,5 @@
         <origin xyz="0 -0.0112 0.15" rpy="0 0 0"/>
         <axis xyz="1 0 0" />
-        <mimic joint="B_Rot->In_1" multiplier="-1" offset="0" />
+        <mimic joint="B_Rot-In_1" multiplier="-1" offset="0" />
     </joint>
     <link name="Join">
@@ -182,5 +180,5 @@
         <axis xyz="1 0 0" />
         <limit lower="-3.14" upper="3.14" effort="30" velocity="1.74533" />
-        <mimic joint="Join->In_2" multiplier="-1" offset="0" />
+        <mimic joint="Join-In_2" multiplier="-1" offset="0" />
     </joint>
     <link name="EE">
